File: kicad/ledregenampel/ledregenampel.kicad_sch (KiCad schematic)
At the start: 102 parts

Commit message: lets call this RC1
Parts:
- added C1, C6: 100nF, Capacitor_SMD:C_0402_1005Metric, symbol Device:C
- added C2, C3, C4, C5: 100uF, Capacitor_SMD:C_1206_3216Metric, symbol Device:C
- added D100, D101, D102, D52, D53, D54, D55, D56, D57, D58, D59, D60, D61, D62, D63, D64, D65, D66, D67, D68, D69, D70, D71, D72, D73, D74, D75, D76, D77, D78, D79, D80, D81, D82, D83, D84, D85, D86, D87, D88, D89, D90, D91, D92, D93, D94, D95, D96, D97, D98, D99: LED Y, LED_SMD:LED_0805_2012Metric, symbol Device:LED
- added D103, D104, D105, D106, D107, D108, D109, D110, D111, D112, D113, D114, D115, D116, D117, D118, D119, D120, D121, D122, D123, D124, D125, D126, D127, D128, D129, D130, D131, D132, D133, D134, D135, D136, D137, D138, D139, D140, D141, D142, D143, D144, D145, D146, D147, D148, D149, D150, D151, D152, D153: LED R, LED_SMD:LED_0805_2012Metric, symbol Device:LED
- added J1: Exp-Conn1, Connector_PinHeader_2.54mm:PinHeader_1x04_P2.54mm_Vertical, symbol Connector:Conn_01x04_Pin
- added J2: Exp-Conn2, Connector_PinHeader_2.54mm:PinHeader_1x01_P2.54mm_Vertical, symbol Connector:Conn_01x01_Pin
- added Q1, Q2, Q3: AO3400A, Package_TO_SOT_SMD:SOT-23, symbol Transistor_FET:AO3400A
- added R100, R101, R102, R103, R104, R105, R106, R107, R108, R109, R110, R111, R112, R113, R114, R115, R116, R117, R118, R119, R120, R121, R122, R123, R124, R125, R126, R127, R128, R129, R130, R131, R132, R133, R134, R135, R136, R137, R138, R139, R140, R141, R142, R143, R144, R145, R146, R147, R148, R149, R150, R151, R152, R153, R52, R53, R54, R55, R56, R57, R58, R59, R60, R61, R62, R63, R64, R65, R66, R67, R68, R69, R70, R71, R72, R73, R74, R75, R76, R77, R78, R79, R80, R81, R82, R83, R84, R85, R86, R87, R88, R89, R90, R91, R92, R93, R94, R95, R96, R97, R98, R99: 150Ω, foxisfrickellibrary:R_0402_modsilkscreen, symbol Device:R
- added R154, R155, R156: 33Ω, foxisfrickellibrary:R_0402_modsilkscreen, symbol Device:R
- added R157, R158, R159: 1MΩ, foxisfrickellibrary:R_0402_modsilkscreen, symbol Device:R
- added U1: Waveshare ESP32-C3 Mini, foxisfrickellibrary:Waveshare_ESP32-C3_Mini, symbol foxisfrickellibrary:Waveshare_ESP32-C3_Mini
- added U2: ~, foxisfrickellibrary:OLED-2.08-inch, symbol foxisfrickellibrary:OLED-2.08inch
- R1, R10, R11, R12, R13, R14, R15, R16, R17, R18, R19, R2, R20, R21, R22, R23, R24, R25, R26, R27, R28, R29, R3, R30, R31, R32, R33, R34, R35, R36, R37, R38, R39, R4, R40, R41, R42, R43, R44, R45, R46, R47, R48, R49, R5, R50, R51, R6, R7, R8, R9: value 110 -> 120Ω
Connections:
- net +5V: now also C2.1, C3.1, C4.1, C5.1, D100.2 (A), D101.2 (A), D102.2 (A), D103.2 (A), D104.2 (A), D105.2 (A), D106.2 (A), D107.2 (A), D108.2 (A), D109.2 (A), D110.2 (A), D111.2 (A), D112.2 (A), D113.2 (A), D114.2 (A), D115.2 (A), D116.2 (A), D117.2 (A), D118.2 (A), D119.2 (A), D120.2 (A), D121.2 (A), D122.2 (A), D123.2 (A), D124.2 (A), D125.2 (A), D126.2 (A), D127.2 (A), D128.2 (A), D129.2 (A), D130.2 (A), D131.2 (A), D132.2 (A), D133.2 (A), D134.2 (A), D135.2 (A), D136.2 (A), D137.2 (A), D138.2 (A), D139.2 (A), D140.2 (A), D141.2 (A), D142.2 (A), D143.2 (A), D144.2 (A), D145.2 (A), D146.2 (A), D147.2 (A), D148.2 (A), D149.2 (A), D150.2 (A), D151.2 (A), D152.2 (A), D153.2 (A), D52.2 (A), D53.2 (A), D54.2 (A), D55.2 (A), D56.2 (A), D57.2 (A), D58.2 (A), D59.2 (A), D60.2 (A), D61.2 (A), D62.2 (A), D63.2 (A), D64.2 (A), D65.2 (A), D66.2 (A), D67.2 (A), D68.2 (A), D69.2 (A), D70.2 (A), D71.2 (A), D72.2 (A), D73.2 (A), D74.2 (A), D75.2 (A), D76.2 (A), D77.2 (A), D78.2 (A), D79.2 (A), D80.2 (A), D81.2 (A), D82.2 (A), D83.2 (A), D84.2 (A), D85.2 (A), D86.2 (A), D87.2 (A), D88.2 (A), D89.2 (A), D90.2 (A), D91.2 (A), D92.2 (A), D93.2 (A), D94.2 (A), D95.2 (A), D96.2 (A), D97.2 (A), D98.2 (A), D99.2 (A), U1.1 (5V)
- net G2MOSFET: now also Q3.3 (D)
- new net: D55.1 (K), R55.1
- new net: D114.1 (K), R114.1
- new net: D117.1 (K), R117.1
- new net: D68.1 (K), R68.1
- new net: D138.1 (K), R138.1
- new net: D123.1 (K), R123.1
- new net: D85.1 (K), R85.1
- new net: D83.1 (K), R83.1
- new net: D81.1 (K), R81.1
- new net: D144.1 (K), R144.1
- new net: D112.1 (K), R112.1
- new net: D58.1 (K), R58.1
- new net: D139.1 (K), R139.1
- new net: D130.1 (K), R130.1
- new net: D149.1 (K), R149.1
- new net: D131.1 (K), R131.1
- new net: D96.1 (K), R96.1
- new net: D111.1 (K), R111.1
- new net: D127.1 (K), R127.1
- new net: D60.1 (K), R60.1
- new net: D64.1 (K), R64.1
- new net: D118.1 (K), R118.1
- new net: D128.1 (K), R128.1
- new net: D57.1 (K), R57.1
- new net: Q2.1 (G), R155.1, R158.1
- new net: J2.1 (Pin_1), U1.10 (GP6)
- new net: D106.1 (K), R106.1
- new net: D105.1 (K), R105.1
- new net: D140.1 (K), R140.1
- new net: D72.1 (K), R72.1
- new net: D94.1 (K), R94.1
- new net: D91.1 (K), R91.1
- new net: D153.1 (K), R153.1
- new net: D89.1 (K), R89.1
- new net: D108.1 (K), R108.1
- new net: D124.1 (K), R124.1
- new net: D120.1 (K), R120.1
- new net: D74.1 (K), R74.1
- new net: D107.1 (K), R107.1
- new net: D100.1 (K), R100.1
- new net: D113.1 (K), R113.1
- new net: D65.1 (K), R65.1
- new net: D103.1 (K), R103.1
- new net: D119.1 (K), R119.1
- new net: D110.1 (K), R110.1
- new net: D79.1 (K), R79.1
- new net: D59.1 (K), R59.1
- new net: D82.1 (K), R82.1
- new net: D148.1 (K), R148.1
- new net: D102.1 (K), R102.1
- new net: D121.1 (K), R121.1
- new net: D134.1 (K), R134.1
- new net: D133.1 (K), R133.1
- new net: D73.1 (K), R73.1
- new net: D67.1 (K), R67.1
- new net: D99.1 (K), R99.1
- new net: D122.1 (K), R122.1
- new net: D137.1 (K), R137.1
- new net: D132.1 (K), R132.1
- new net: D71.1 (K), R71.1
- new net: Q1.1 (G), R154.1, R157.1
- new net: D75.1 (K), R75.1
- new net: D53.1 (K), R53.1
- new net: D56.1 (K), R56.1
- new net: D90.1 (K), R90.1
- new net: Q3.1 (G), R156.1, R159.1
- new net: D92.1 (K), R92.1
- new net: D78.1 (K), R78.1
- new net: D97.1 (K), R97.1
- new net: D87.1 (K), R87.1
- new net: D62.1 (K), R62.1
- new net: D116.1 (K), R116.1
- new net: D150.1 (K), R150.1
- new net: D146.1 (K), R146.1
- new net: D95.1 (K), R95.1
- new net: D141.1 (K), R141.1
- new net: D52.1 (K), R52.1
- new net: D125.1 (K), R125.1
- new net: D147.1 (K), R147.1
- new net: D80.1 (K), R80.1
- new net: D93.1 (K), R93.1
- new net: D145.1 (K), R145.1
- new net: D143.1 (K), R143.1
- new net: D98.1 (K), R98.1
- new net: D104.1 (K), R104.1
- new net: D69.1 (K), R69.1
- new net: D152.1 (K), R152.1
- new net: D70.1 (K), R70.1
- new net: D142.1 (K), R142.1
- new net: D129.1 (K), R129.1
- new net: D63.1 (K), R63.1
- new net: D135.1 (K), R135.1
- new net: D88.1 (K), R88.1
- new net: D77.1 (K), R77.1
- new net: R154.2, U1.11 (GP7)
- new net: D54.1 (K), R54.1
- new net: D109.1 (K), R109.1
- new net: D115.1 (K), R115.1
- new net: D61.1 (K), R61.1
- new net: D84.1 (K), R84.1
- new net: D86.1 (K), R86.1
- new net: D66.1 (K), R66.1
- new net: D136.1 (K), R136.1
- new net: R156.2, U1.12 (GP8)
- new net: D151.1 (K), R151.1
- new net: J1.1 (Pin_1), U1.6 (GP2)
- new net: J1.2 (Pin_2), U1.7 (GP3)
- new net: J1.3 (Pin_3), U1.8 (GP4)
- new net: J1.4 (Pin_4), U1.9 (GP5)
- new net: D101.1 (K), R101.1
- new net: D76.1 (K), R76.1
- new net: D126.1 (K), R126.1
- new net: U1.4 (GP0), U2.3 (SCL)
- new net: U1.5 (GP1), U2.4 (SDA)
- new net: R155.2, U1.13 (GP9)
- new net +3V3: C1.1, C6.2, U1.3 (3V3), U2.2 (VCC)
- new net GND: C1.2, C2.2, C3.2, C4.2, C5.2, C6.1, Q1.2 (S), Q2.2 (S), Q3.2 (S), R157.2, R158.2, R159.2, U1.2 (GND), U2.1 (GND)
- new net R2MOSFET: Q1.3 (D), R103.2, R104.2, R105.2, R106.2, R107.2, R108.2, R109.2, R110.2, R111.2, R112.2, R113.2, R114.2, R115.2, R116.2, R117.2, R118.2, R119.2, R120.2, R121.2, R122.2, R123.2, R124.2, R125.2, R126.2, R127.2, R128.2, R129.2, R130.2, R131.2, R132.2, R133.2, R134.2, R135.2, R136.2, R137.2, R138.2, R139.2, R140.2, R141.2, R142.2, R143.2, R144.2, R145.2, R146.2, R147.2, R148.2, R149.2, R150.2, R151.2, R152.2, R153.2
- new net Y2MOSFET: Q2.3 (D), R100.2, R101.2, R102.2, R52.2, R53.2, R54.2, R55.2, R56.2, R57.2, R58.2, R59.2, R60.2, R61.2, R62.2, R63.2, R64.2, R65.2, R66.2, R67.2, R68.2, R69.2, R70.2, R71.2, R72.2, R73.2, R74.2, R75.2, R76.2, R77.2, R78.2, R79.2, R80.2, R81.2, R82.2, R83.2, R84.2, R85.2, R86.2, R87.2, R88.2, R89.2, R90.2, R91.2, R92.2, R93.2, R94.2, R95.2, R96.2, R97.2, R98.2, R99.2
Other:
- note added: "GP10 in use by onboard WS2812"
- note added: "do not use GP18-21 - very restricted functionality"

Commit message: mostly more labelling
Parts:
- added J3: I2Cout, Connector_PinHeader_2.54mm:PinHeader_1x02_P2.54mm_Vertical, symbol Connector:Conn_01x02_Pin
- added J4: Conn_5V, Connector_PinHeader_2.54mm:PinHeader_1x02_P2.54mm_Vertical, symbol Connector_Generic:Conn_01x02
- added J5: Conn_3V3, Connector_PinHeader_2.54mm:PinHeader_1x02_P2.54mm_Vertical, symbol Connector:Conn_01x02_Pin
- J1, J2, U1: now left out of the parts list
- U2: value ~ -> OLED 2.08 inch; now left out of the parts list
Connections:
- net +3V3: now also J5.1 (Pin_1)
- net +5V: now also J4.1 (Pin_1)
- net GND: now also J4.2 (Pin_2), J5.2 (Pin_2)
- net at U1.4 (GP0), U2.3 (SCL): now also J3.1 (Pin_1)
- net at U1.5 (GP1), U2.4 (SDA): now also J3.2 (Pin_2)
